Commit message: Dif if moving

File: catkin_ws/src/fre_task4_description/urdf/fre_robot_minimal.urdf.xacro (robot description, xacro)
@@ -9,4 +9,9 @@
   <xacro:property name="wheel_radius" value="0.12"/>
   <xacro:property name="wheel_width"  value="0.06"/>
+  <xacro:property name="wheel_separation" value="0.76"/>
+  <!-- Robot is lifted so the chassis is not touching the ground.
+       Wheel center height = wheel_radius = 0.12 m.
+       base_link center height = 0.275 m.
+       Wheel joint z relative to base_link = 0.12 - 0.275 = -0.155 m. -->
   <!-- ===================== -->
   <!-- base_footprint         -->
@@ -16,5 +21,5 @@
     <parent link="base_footprint"/>
     <child link="base_link"/>
-    <origin xyz="0 0 0.175" rpy="0 0 0"/>
+    <origin xyz="0 0 0.275" rpy="0 0 0"/>
   </joint>
   <!-- ===================== -->
@@ -40,7 +45,75 @@
       <origin xyz="0 0 0"/>
       <mass value="25.0"/>
-      <inertia ixx="1.5" ixy="0" ixz="0" iyy="1.5" iyz="0" izz="1.5"/>
-    </inertial>
-  </link>
+      <inertia ixx="1.5" ixy="0" ixz="0"
+               iyy="1.5" iyz="0"
+               izz="1.5"/>
+    </inertial>
+  </link>
+  <!-- ===================== -->
+  <!-- left wheel             -->
+  <!-- ===================== -->
+  <link name="left_wheel_link">
+    <visual>
+      <origin xyz="0 0 0" rpy="1.5708 0 0"/>
+      <geometry>
+        <cylinder radius="${wheel_radius}" length="${wheel_width}"/>
+      </geometry>
+      <material name="black">
+        <color rgba="0.02 0.02 0.02 1.0"/>
+      </material>
+    </visual>
+    <collision>
+      <origin xyz="0 0 0" rpy="1.5708 0 0"/>
+      <geometry>
+        <cylinder radius="${wheel_radius}" length="${wheel_width}"/>
+      </geometry>
+    </collision>
+    <inertial>
+      <origin xyz="0 0 0"/>
+      <mass value="1.0"/>
+      <inertia ixx="0.01" ixy="0" ixz="0"
+               iyy="0.01" iyz="0"
+               izz="0.01"/>
+    </inertial>
+  </link>
+  <joint name="left_wheel_joint" type="continuous">
+    <parent link="base_link"/>
+    <child link="left_wheel_link"/>
+    <origin xyz="0.0 0.38 -0.155" rpy="0 0 0"/>
+    <axis xyz="0 1 0"/>
+  </joint>
+  <!-- ===================== -->
+  <!-- right wheel            -->
+  <!-- ===================== -->
+  <link name="right_wheel_link">
+    <visual>
+      <origin xyz="0 0 0" rpy="1.5708 0 0"/>
+      <geometry>
+        <cylinder radius="${wheel_radius}" length="${wheel_width}"/>
+      </geometry>
+      <material name="black">
+        <color rgba="0.02 0.02 0.02 1.0"/>
+      </material>
+    </visual>
+    <collision>
+      <origin xyz="0 0 0" rpy="1.5708 0 0"/>
+      <geometry>
+        <cylinder radius="${wheel_radius}" length="${wheel_width}"/>
+      </geometry>
+    </collision>
+    <inertial>
+      <origin xyz="0 0 0"/>
+      <mass value="1.0"/>
+      <inertia ixx="0.01" ixy="0" ixz="0"
+               iyy="0.01" iyz="0"
+               izz="0.01"/>
+    </inertial>
+  </link>
+  <joint name="right_wheel_joint" type="continuous">
+    <parent link="base_link"/>
+    <child link="right_wheel_link"/>
+    <origin xyz="0.0 -0.38 -0.155" rpy="0 0 0"/>
+    <axis xyz="0 1 0"/>
+  </joint>
   <!-- ===================== -->
   <!-- lidar                  -->
@@ -55,4 +128,16 @@
       </material>
     </visual>
+    <collision>
+      <geometry>
+        <cylinder radius="0.05" length="0.06"/>
+      </geometry>
+    </collision>
+    <inertial>
+      <origin xyz="0 0 0"/>
+      <mass value="0.2"/>
+      <inertia ixx="0.001" ixy="0" ixz="0"
+               iyy="0.001" iyz="0"
+               izz="0.001"/>
+    </inertial>
   </link>
   <joint name="base_link_to_lidar" type="fixed">
@@ -73,4 +158,16 @@
       </material>
     </visual>
+    <collision>
+      <geometry>
+        <box size="0.08 0.03 0.03"/>
+      </geometry>
+    </collision>
+    <inertial>
+      <origin xyz="0 0 0"/>
+      <mass value="0.1"/>
+      <inertia ixx="0.0005" ixy="0" ixz="0"
+               iyy="0.0005" iyz="0"
+               izz="0.0005"/>
+    </inertial>
   </link>
   <joint name="base_link_to_front_camera" type="fixed">
@@ -83,5 +180,5 @@
     <parent link="front_camera_link"/>
     <child link="front_camera_optical_frame"/>
-    <!-- ROS optical frame: z forward, x right, y down -->
+    <!-- ROS optical frame convention: z forward, x right, y down -->
     <origin xyz="0 0 0" rpy="-1.5708 0 -1.5708"/>
   </joint>
@@ -98,4 +195,16 @@
       </material>
     </visual>
+    <collision>
+      <geometry>
+        <box size="0.08 0.03 0.03"/>
+      </geometry>
+    </collision>
+    <inertial>
+      <origin xyz="0 0 0"/>
+      <mass value="0.1"/>
+      <inertia ixx="0.0005" ixy="0" ixz="0"
+               iyy="0.0005" iyz="0"
+               izz="0.0005"/>
+    </inertial>
   </link>
   <joint name="base_link_to_down_camera" type="fixed">
@@ -111,5 +220,5 @@
   </joint>
   <!-- ===================== -->
-  <!-- treatment tool / nozzle -->
+  <!-- treatment tool/nozzle  -->
   <!-- ===================== -->
   <link name="treatment_tool_link">
@@ -122,4 +231,16 @@
       </material>
     </visual>
+    <collision>
+      <geometry>
+        <cylinder radius="0.025" length="0.12"/>
+      </geometry>
+    </collision>
+    <inertial>
+      <origin xyz="0 0 0"/>
+      <mass value="0.1"/>
+      <inertia ixx="0.0005" ixy="0" ixz="0"
+               iyy="0.0005" iyz="0"
+               izz="0.0005"/>
+    </inertial>
   </link>
   <joint name="base_link_to_treatment_tool" type="fixed">
@@ -129,35 +250,59 @@
   </joint>
   <!-- ===================== -->
-  <!-- wheels, visual only    -->
-  <!-- ===================== -->
-  <link name="left_wheel_link">
-    <visual>
-      <origin xyz="0 0 0" rpy="1.5708 0 0"/>
-      <geometry>
-        <cylinder radius="${wheel_radius}" length="${wheel_width}"/>
-      </geometry>
-      <material name="black">
-        <color rgba="0.02 0.02 0.02 1.0"/>
-      </material>
-    </visual>
-  </link>
-  <joint name="base_link_to_left_wheel" type="fixed">
-    <parent link="base_link"/>
-    <child link="left_wheel_link"/>
-    <origin xyz="0.0 0.38 -0.10" rpy="0 0 0"/>
-  </joint>
-  <link name="right_wheel_link">
-    <visual>
-      <origin xyz="0 0 0" rpy="1.5708 0 0"/>
-      <geometry>
-        <cylinder radius="${wheel_radius}" length="${wheel_width}"/>
-      </geometry>
-      <material name="black"/>
-    </visual>
-  </link>
-  <joint name="base_link_to_right_wheel" type="fixed">
-    <parent link="base_link"/>
-    <child link="right_wheel_link"/>
-    <origin xyz="0.0 -0.38 -0.10" rpy="0 0 0"/>
-  </joint>
+  <!-- Gazebo visual/friction -->
+  <!-- ===================== -->
+  <gazebo reference="base_link">
+    <material>Gazebo/DarkGrey</material>
+  </gazebo>
+  <gazebo reference="left_wheel_link">
+    <material>Gazebo/Black</material>
+    <mu1>5.0</mu1>
+    <mu2>5.0</mu2>
+    <kp>1000000.0</kp>
+    <kd>10.0</kd>
+  </gazebo>
+  <gazebo reference="right_wheel_link">
+    <material>Gazebo/Black</material>
+    <mu1>5.0</mu1>
+    <mu2>5.0</mu2>
+    <kp>1000000.0</kp>
+    <kd>10.0</kd>
+  </gazebo>
+  <gazebo reference="lidar_link">
+    <material>Gazebo/Blue</material>
+  </gazebo>
+  <gazebo reference="front_camera_link">
+    <material>Gazebo/Green</material>
+  </gazebo>
+  <gazebo reference="down_camera_link">
+    <material>Gazebo/Yellow</material>
+  </gazebo>
+  <gazebo reference="treatment_tool_link">
+    <material>Gazebo/Red</material>
+  </gazebo>
+  <!-- ===================== -->
+  <!-- Differential drive     -->
+  <!-- ===================== -->
+  <gazebo>
+    <plugin name="fre_diff_drive" filename="libgazebo_ros_diff_drive.so">
+      <legacyMode>false</legacyMode>
+      <leftJoint>left_wheel_joint</leftJoint>
+      <rightJoint>right_wheel_joint</rightJoint>
+      <wheelSeparation>${wheel_separation}</wheelSeparation>
+      <wheelDiameter>${2.0 * wheel_radius}</wheelDiameter>
+      <wheelTorque>80</wheelTorque>
+      <wheelAcceleration>5.0</wheelAcceleration>
+      <commandTopic>cmd_vel</commandTopic>
+      <odometryTopic>odom</odometryTopic>
+      <odometryFrame>odom</odometryFrame>
+      <robotBaseFrame>base_footprint</robotBaseFrame>
+      <publishTf>true</publishTf>
+      <publishOdomTF>true</publishOdomTF>
+      <publishWheelTF>false</publishWheelTF>
+      <publishWheelJointState>true</publishWheelJointState>
+      <odometrySource>world</odometrySource>
+      <updateRate>50</updateRate>
+      <rosDebugLevel>na</rosDebugLevel>
+    </plugin>
+  </gazebo>
 </robot>
